File: boards/main.brd (EAGLE design)
At the start: 157 x 20 mm, 47 parts, among them CON2 MINI-USB-, IC1 74595AP, IC2 STM32F103CBT6, IC3 74595AP, IC4 TAR5SB33, Q1 FA-238V

Commit message: update board design
Parts:
- added IC5: 74VHC541A, IC_Robotech:TSSOP20
- moved R3 1.02 mm to (38.9, 17.8)
- moved C3 0.76 mm to (40.6, 6.60)
Connections:
- new net CLK_BUF: IC1.11, IC3.11, IC5.17
- new net DATA_IN_BUF: IC1.14, IC5.18
- new net RATCH_BUF: IC1.12, IC3.12, IC5.16
- net +5V: now also IC5.20
- net CLK: now also IC5.3; no longer IC1.11, IC3.11
- net DATA_IN: now also IC5.2; no longer IC1.14
- net GND: now also IC5.1, IC5.10, IC5.19, IC5.5, IC5.6, IC5.7, IC5.8, IC5.9
- net RATCH: now also IC5.4; no longer IC1.12, IC3.12
Routing:
- net RATCH_BUF: track 0.00 -> 108.7 mm
- net CLK_BUF: track 0.00 -> 102.9 mm, vias 0 -> 1
- net CLK: track 115.4 -> 22.1 mm, vias 3 -> 0
- net RATCH: track 115.0 -> 25.3 mm
- net +5V: track 159.2 -> 185.0 mm
- net DATA_IN: track 40.8 -> 19.8 mm
- net DATA_IN_BUF: track 0.00 -> 19.9 mm
- net DATA_OUT: track 0.00 -> 8.29 mm
- net N$17: track 49.4 -> 46.4 mm
- net N$16: track 69.5 -> 67.1 mm
- net +3V3: track 82.1 -> 80.5 mm
- net N$18: track 35.8 -> 34.5 mm
- net N$5: track 4.07 -> 4.94 mm
- net N$21: track 11.6 -> 10.8 mm
- net N$28: track 26.0 -> 26.6 mm
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- added copper zone on layer 1, net +5V
- added copper zone on layer 16, net CLK_BUF
- added copper zone on layer 1, net DATA_OUT
- added copper zone on layer 16, net NC
- added copper zone on layer 1, net RATCH_BUF
Other:
- board text added: "SWCLK"
- board text added: "SWDIO"
