File: boards/main.sch (EAGLE design)
At the start: 47 parts, among them CON2 MINI-USB-, IC1 74595AP, IC2 STM32F103CBT6, IC3 74595AP, IC4 TAR5SB33, Q1 FA-238V

Commit message: update board design
Parts:
- added IC5: 74VHC541A, IC_Robotech:74VHC541A
Connections:
- new net CLK_BUF: IC1G$1.SCLK, IC3G$1.SCLK, IC5G$1.Y2
- new net DATA_IN_BUF: IC1G$1.SER, IC5G$1.Y1
- new net RATCH_BUF: IC1G$1.RCLK, IC3G$1.RCLK, IC5G$1.Y3
- net CLK: now also IC5G$1.A2; no longer IC1G$1.SCLK, IC3G$1.SCLK
- net DATA_IN: now also IC5G$1.A1; no longer IC1G$1.SER
- net GND: now also IC5G$1.!OE1, IC5G$1.!OE2, IC5G$1.A4, IC5G$1.A5, IC5G$1.A6, IC5G$1.A7, IC5G$1.A8
- net RATCH: now also IC5G$1.A3; no longer IC1G$1.RCLK, IC3G$1.RCLK
